File: board/board.kicad_pcb (KiCad board)
At the start: 2 copper layers, 21 x 13 mm, 1 part

Commit message: initial
Parts:
- added C1: 1uF, Capacitor_SMD:C_0603_1608Metric, F.Cu at (151.0, 93.5)
- added C2: 10uF, Capacitor_SMD:C_0603_1608Metric, F.Cu at (151.0, 92.0)
- added J1: 002_SPI, on_edge:on_edge_2x05_device, F.Cu at (140.0, 96.5)
- added J2: 007_ADC, on_edge:on_edge_2x05_host, F.Cu at (161.0, 96.5)
- added U1: DAC121S101, Package_TO_SOT_SMD:SOT-23-6, F.Cu at (150.5, 96.0)
- LOGO1: moved to B.Cu
- moved LOGO1 2.21 mm to (150.7, 96.9), turned to 180 degrees
Routing:
- net /dac/VDD: track 0.00 -> 26.4 mm, vias 0 -> 3
- net GND: track 0.00 -> 21.3 mm, vias 0 -> 26
- net Net-(J1-Pad9): track 0.00 -> 16.2 mm
- net /dac/~{SYNC}: track 0.00 -> 10.4 mm, vias 0 -> 1
- net /dac/SCLK: track 0.00 -> 8.05 mm
- net /dac/MOSI: track 0.00 -> 7.24 mm
- net /dac/out: track 0.00 -> 7.20 mm
- added copper zone on B.Cu, net GND
- added copper zone on F.Cu, net GND
Other:
- outline, holes or cut-outs redrawn
- board text added: "osf.002"
- board text added: "osf.007"
- board text added: "osf.b125.v1.0"
